File: hardware/suma-v-0-rev-b/suma-v-0-rev-b.kicad_pcb (KiCad board)
At the start: 2 copper layers, 25 x 100 mm, 20 parts, among them J1 AudioJack2_SwitchT, J2 AudioJack2_SwitchT, J3 AudioJack2_SwitchT, J4 Conn_02x05_Odd_Even, J5 AudioJack2_SwitchT, U1 TL072

Commit message: añadidos vdc
Connections:
- net Net-(D1-A) renamed +VDC
- net Net-(D2-K) renamed -VDC
Changed lines of the file:
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@@
 			(size 1.48 1.4)
 			(layers "F.Cu" "F.Mask" "F.Paste")
-			(net "Net-(D2-K)")
+			(net "-VDC")
 			(pinfunction "K_1")
 			(pintype "passive")
@@
 			(size 1.48 1.4)
 			(layers "F.Cu" "F.Mask" "F.Paste")
-			(net "Net-(D1-A)")
+			(net "+VDC")
 			(pinfunction "A_2")
 			(pintype "passive")
@@
 			(remove_unused_layers no)
 			(roundrect_rratio 0.125)
-			(net "Net-(D2-K)")
+			(net "-VDC")
 			(pinfunction "Pin_1_1")
 			(pintype "passive")
@@
 			(layers "*.Cu" "*.Mask")
 			(remove_unused_layers no)
-			(net "Net-(D2-K)")
+			(net "-VDC")
 			(pinfunction "Pin_2_2")
 			(pintype "passive")
@@
 			(layers "*.Cu" "*.Mask")
 			(remove_unused_layers no)
-			(net "Net-(D1-A)")
+			(net "+VDC")
 			(pinfunction "Pin_9_9")
 			(pintype "passive")
@@
 			(layers "*.Cu" "*.Mask")
 			(remove_unused_layers no)
-			(net "Net-(D1-A)")
+			(net "+VDC")
 			(pinfunction "Pin_10_10")
 			(pintype "passive")
@@
 	)
 	(segment
-		(start 37.6 34.3)
-		(end 37.6 37.54)
-		(width 0.8)
-		(layer "F.Cu")
-		(net "Net-(D2-K)")
-	)
-	(segment
-		(start 37.6 37.54)
-		(end 37.6 43.81)
-		(width 0.8)
-		(layer "F.Cu")
-		(net "Net-(D2-K)")
-	)
-	(segment
-		(start 37.6 43.81)
-		(end 37.41 44)
-		(width 0.8)
-		(layer "F.Cu")
-		(net "Net-(D2-K)")
-	)
-	(segment
 		(start 38 55.312)
 		(end 39.188 56.5)
@@
 	)
 	(segment
-		(start 48 37.3)
-		(end 47.76 37.54)
-		(width 0.8)
-		(layer "F.Cu")
-		(net "Net-(D1-A)")
-	)
-	(segment
-		(start 48 34.54)
-		(end 48 37.3)
-		(width 0.8)
-		(layer "F.Cu")
-		(net "Net-(D1-A)")
-	)
-	(segment
-		(start 47.59 44)
-		(end 47.59 37.71)
-		(width 0.8)
-		(layer "F.Cu")
-		(net "Net-(D1-A)")
-	)
-	(segment
-		(start 47.76 34.3)
-		(end 48 34.54)
-		(width 0.8)
-		(layer "F.Cu")
-		(net "Net-(D1-A)")
-	)
-	(segment
-		(start 47.59 37.71)
-		(end 47.76 37.54)
-		(width 0.8)
-		(layer "F.Cu")
-		(net "Net-(D1-A)")
-	)
-	(segment
-		(start 47.76 43.83)
-		(end 47.59 44)
-		(width 0.8)
-		(layer "F.Cu")
-		(net "Net-(D1-A)")
-	)
-	(segment
 		(start 36 52.5)
 		(end 35 51.5)
@@
 		(net "Net-(R1-Pad1)")
 	)
+	(segment
+		(start 48 37.3)
+		(end 47.76 37.54)
+		(width 0.8)
+		(layer "F.Cu")
+		(net "+VDC")
+	)
+	(segment
+		(start 48 34.54)
+		(end 48 37.3)
+		(width 0.8)
+		(layer "F.Cu")
+		(net "+VDC")
+	)
+	(segment
+		(start 47.59 44)
+		(end 47.59 37.71)
+		(width 0.8)
+		(layer "F.Cu")
+		(net "+VDC")
+	)
+	(segment
+		(start 47.76 34.3)
+		(end 48 34.54)
+		(width 0.8)
+		(layer "F.Cu")
+		(net "+VDC")
+	)
+	(segment
+		(start 47.59 37.71)
+		(end 47.76 37.54)
+		(width 0.8)
+		(layer "F.Cu")
+		(net "+VDC")
+	)
+	(segment
+		(start 47.76 43.83)
+		(end 47.59 44)
+		(width 0.8)
+		(layer "F.Cu")
+		(net "+VDC")
+	)
+	(segment
+		(start 37.6 34.3)
+		(end 37.6 37.54)
+		(width 0.8)
+		(layer "F.Cu")
+		(net "-VDC")
+	)
+	(segment
+		(start 37.6 37.54)
+		(end 37.6 43.81)
+		(width 0.8)
+		(layer "F.Cu")
+		(net "-VDC")
+	)
+	(segment
+		(start 37.6 43.81)
+		(end 37.41 44)
+		(width 0.8)
+		(layer "F.Cu")
+		(net "-VDC")
+	)
 	(zone
